Commit message: add apf and edit k

File: segway_v3/segway_description/urdf/RMP_220/rmp.urdf.xacro (robot description, xacro)
@@ -296,4 +296,36 @@
     <origin xyz="-0.005 0.02 1.245" rpy="0.07 0 0" />
   </xacro:VLP-16>
+    <gazebo reference="velodyne">
+    <material>Gazebo/FlatBlack</material>
+    <sensor type="ray" name="lds_lfcd_sensor">
+      <pose>0 0 0 0 0 0</pose>
+      <visualize>False</visualize>
+      <update_rate>10</update_rate>
+      <ray>
+        <scan>
+          <horizontal>
+            <samples>1024</samples>
+            <resolution>1</resolution>
+            <min_angle>0.0</min_angle>
+            <max_angle>6.28319</max_angle>
+          </horizontal>
+        </scan>
+        <range>
+          <min>0.1</min>
+          <max>10</max>
+          <resolution>0.015</resolution>
+        </range>
+        <noise>
+          <type>gaussian</type>
+          <mean>0.0</mean>
+          <stddev>0.01</stddev>
+        </noise>
+      </ray>
+      <plugin name="gazebo_ros_lds_lfcd_controller" filename="libgazebo_ros_laser.so">
+        <topicName>scan</topicName>
+        <frameName>base_scan</frameName>
+      </plugin>
+    </sensor>
+  </gazebo>
   <!-- # ZED ###################################################################################### -->
    <xacro:include filename="$(find zed_description)/urdf/zed_descr.urdf.xacro"/>
